Commit message: Load G1 model on RVIZ

File: ros2_ws/src/hardware/hardware_bringup/urdf/g1_23dof.urdf (robot description, URDF)
Before this commit: robot g1_23dof, 34 links, 33 joints
Links:
- link head_link: geometry collision mesh filename=package://hardware_bringup/meshes/head_link.STL; visual mesh filename=package://hardware_bringup/meshes/head_link.STL
- link left_ankle_pitch_link: geometry collision mesh filename=package://hardware_bringup/meshes/left_ankle_pitch_link.STL; visual mesh filename=package://hardware_bringup/meshes/left_ankle_pitch_link.STL
- link left_ankle_roll_link: geometry collision sphere radius=0.005; collision sphere radius=0.005
- link left_elbow_link: geometry collision mesh filename=package://hardware_bringup/meshes/left_elbow_link.STL; visual mesh filename=package://hardware_bringup/meshes/left_elbow_link.STL
- link left_hip_pitch_link: geometry collision mesh filename=package://hardware_bringup/meshes/left_hip_pitch_link.STL; visual mesh filename=package://hardware_bringup/meshes/left_hip_pitch_link.STL
- link left_hip_roll_link: geometry collision mesh filename=package://hardware_bringup/meshes/left_hip_roll_link.STL; visual mesh filename=package://hardware_bringup/meshes/left_hip_roll_link.STL
- link left_hip_yaw_link: geometry collision mesh filename=package://hardware_bringup/meshes/left_hip_yaw_link.STL; visual mesh filename=package://hardware_bringup/meshes/left_hip_yaw_link.STL
- link left_knee_link: geometry collision mesh filename=package://hardware_bringup/meshes/left_knee_link.STL; visual mesh filename=package://hardware_bringup/meshes/left_knee_link.STL
- link left_shoulder_pitch_link: geometry collision cylinder length=0.05 radius=0.03; visual mesh filename=package://hardware_bringup/meshes/left_shoulder_pitch_link.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
- link left_shoulder_roll_link: geometry collision cylinder length=0.03 radius=0.03; visual mesh filename=package://hardware_bringup/meshes/left_shoulder_roll_link.S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
- link left_shoulder_yaw_link: geometry collision mesh filename=package://hardware_bringup/meshes/left_shoulder_yaw_link.STL; visual mesh filename=package://hardware_bringup/meshes/left_shoulder_yaw_link.STL
- link left_wrist_roll_rubber_hand: geometry collision mesh filename=package://hardware_bringup/meshes/left_wrist_roll_rubber_ha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; visual mesh filename=package://hardware_bringup/meshes/left_wrist_roll_rubber_ha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
- link logo_link: geometry collision mesh filename=package://hardware_bringup/meshes/logo_link.STL; visual mesh filename=package://hardware_bringup/meshes/logo_link.STL
- link pelvis: geometry visual mesh filename=package://hardware_bringup/meshes/pelvis.STL
- link pelvis_contour_link: geometry collision mesh filename=package://hardware_bringup/meshes/pelvis_contour_link.STL; visual mesh filename=package://hardware_bringup/meshes/pelvis_contour_link.STL
- link right_ankle_pitch_link: geometry collision mesh filename=package://hardware_bringup/meshes/right_ankle_pitch_link.STL; visual mesh filename=package://hardware_bringup/meshes/right_ankle_pitch_link.STL
- link right_ankle_roll_link: geometry collision sphere radius=0.005; collision sphere radius=0.005
- link right_elbow_link: geometry collision mesh filename=package://hardware_bringup/meshes/right_elbow_link.STL; visual mesh filename=package://hardware_bringup/meshes/right_elbow_link.STL
- link right_hip_pitch_link: geometry collision mesh filename=package://hardware_bringup/meshes/right_hip_pitch_link.STL; visual mesh filename=package://hardware_bringup/meshes/right_hip_pitch_link.STL
- link right_hip_roll_link: geometry collision mesh filename=package://hardware_bringup/meshes/right_hip_roll_link.STL; visual mesh filename=package://hardware_bringup/meshes/right_hip_roll_link.STL
- link right_hip_yaw_link: geometry collision mesh filename=package://hardware_bringup/meshes/right_hip_yaw_link.STL; visual mesh filename=package://hardware_bringup/meshes/right_hip_yaw_link.STL
- link right_knee_link: geometry collision mesh filename=package://hardware_bringup/meshes/right_knee_link.STL; visual mesh filename=package://hardware_bringup/meshes/right_knee_link.STL
- link right_shoulder_pitch_link: geometry collision cylinder length=0.05 radius=0.03; visual mesh filename=package://hardware_bringup/meshes/right_shoulder_pitch_link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
- link right_shoulder_roll_link: geometry collision cylinder length=0.03 radius=0.03; visual mesh filename=package://hardware_bringup/meshes/right_shoulder_roll_link.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
- link right_shoulder_yaw_link: geometry collision mesh filename=package://hardware_bringup/meshes/right_shoulder_yaw_link.S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; visual mesh filename=package://hardware_bringup/meshes/right_shoulder_yaw_link.S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
- link right_wrist_roll_rubber_hand: geometry collision mesh filename=package://hardware_bringup/meshes/right_wrist_roll_rubber_h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; visual mesh filename=package://hardware_bringup/meshes/right_wrist_roll_rubber_h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
- link torso_link: geometry collision mesh filename=package://hardware_bringup/meshes/torso_link.STL; visual mesh filename=package://hardware_bringup/meshes/torso_link.STL
- link waist_support_link: geometry collision mesh filename=package://hardware_bringup/meshes/waist_support_link.STL; visual mesh filename=package://hardware_bringup/meshes/waist_support_link.STL
- link waist_yaw_fixed_link: geometry visual mesh filename=package://hardware_bringup/meshes/waist_yaw_link.STL
